Commit message: Add colision and inertial tags, Add lidar to urdf

File: src/puzzlebot_ros2/puzzlebot_description/urdf/puzzlebot.urdf.xacro (robot description, xacro)
@@ -2,8 +2,15 @@
 <robot xmlns:xacro="http://www.ros.org/wiki/xacro" name="puzzlebot">
     <xacro:arg name="prefix" default="" />
+    <!-- INERTIAL MACROS AND MATERIALS -->
+    <xacro:include filename="$(find puzzlebot_description)/urdf/misc/macros.xacro"/>
+    <xacro:include filename="$(find puzzlebot_description)/urdf/misc/materials.xacro"/>
     <!-- LINKS AND JOINTS BASE AND WHEELS -->
     <xacro:include filename="$(find puzzlebot_description)/urdf/puzzlebot_core.xacro"/>
+    <!-- LIDAR LINKS AND JOINTS -->
+    <xacro:include filename="$(find puzzlebot_description)/urdf/lidar.xacro"/>
     <!-- CONTROL W/GAZEBO -->
     <xacro:include filename="$(find puzzlebot_description)/urdf/puzzlebot_control.xacro"/>
+    <xacro:puzzlebot_core prefix="$(arg prefix)"/>
+    <xacro:rpi_lidar_sensor prefix="$(arg prefix)"/>
     <xacro:puzzlebot_control prefix="$(arg prefix)"/>
 </robot>

File: src/puzzlebot_ros2/puzzlebot_description/urdf/puzzlebot_control.xacro (robot description, xacro)
@@ -7,5 +7,5 @@
                 <render_engine>ogre2</render_engine>
             </plugin>
-            <plugin filename="gz-sim-diff-drive-systems"
+            <plugin filename="gz-sim-diff-drive-system"
             name="gz::sim::systems::DiffDrive">
                 <left_joint>${prefix}left_wheel_joint</left_joint>

File: src/puzzlebot_ros2/puzzlebot_description/urdf/puzzlebot_core.xacro (robot description, xacro)
@@ -1,74 +1,107 @@
 <?xml version="1.0"?>
 <robot xmlns:xacro="http://www.ros.org/wiki/xacro">
-    <!-- BASE FOOTPRINT -->
-   <link name="base_footprint"></link>
-    <!-- BASE LINK -->
-   <link name="base_link">
-        <visual>
-            <geometry>
-                <mesh filename="package://puzzlebot_description/meshes/Puzzlebot_Jetson_Lidar_Edition_Base.stl"/>
-            </geometry>
-            <material name="yellow">
-                <color rgba="0.8 0.8 0.05 1.0"/>
-            </material>
-        </visual>
-    </link>
-    <joint name="base_link_joint" type="fixed">
-        <origin xyz="0.0 0.0 0.05" rpy="0.0 0.0 0.0"/>
-        <parent link="base_footprint"/>
-        <child link="base_link"/>
-    </joint>
-    <!-- LEFT WHEEL -->
-    <link name="left_wheel_link">
-        <visual>
-            <origin rpy="1.57 0.0 0.0"/>
-            <geometry>
-                <mesh filename="package://puzzlebot_description/meshes/Puzzlebot_Wheel.stl"/>
-            </geometry>
-            <material name="yellow">
-                <color rgba="0.8 0.8 0.05 1.0"/>
-            </material>
-        </visual>
-    </link>
-    <joint name="left_wheel_joint" type="continuous">
-        <parent link="base_link"/>
-        <child link="left_wheel_link"/>
-        <origin xyz="0.052 0.095 -0.0025"/>
-        <axis xyz="0.0 1.0 0.0"/>
-    </joint>
-    <!-- RIGHT WHEEL -->
-    <link name="right_wheel_link">
-        <visual>
-            <origin rpy="-1.57 0.0 0.0"/>
-            <geometry>
-                <mesh filename="package://puzzlebot_description/meshes/Puzzlebot_Wheel.stl"/>
-            </geometry>
-            <material name="yellow">
-                <color rgba="0.8 0.8 0.05 1.0"/>
-            </material>
-        </visual>
-    </link>
-    <joint name="right_wheel_joint" type="continuous">
-        <parent link="base_link"/>
-        <child link="right_wheel_link"/>
-        <origin xyz="0.052 -0.095 -0.0025"/>
-        <axis xyz="0.0 1.0 0.0"/>
-    </joint>
-    <!-- CASTER  WHEEL -->
-    <link name="caster_link">
-        <visual>
-            <origin xyz="0.0 0.0 -0.015"/>
-            <geometry>
-                <mesh filename="package://puzzlebot_description/meshes/Puzzlebot_Caster_Wheel.stl"/>
-            </geometry>
-            <material name="yellow">
-                <color rgba="0.8 0.8 0.05 1.0"/>
-            </material>
-        </visual>
-    </link>
-    <joint name="caster_joint" type="fixed">
-        <parent link="base_link"/>
-        <child link="caster_link"/>
-        <origin xyz="-0.095 0.0 -0.03"/>
-    </joint>
+    <xacro:macro name="puzzlebot_core" params="prefix">
+        <!-- BASE FOOTPRINT -->
+        <link name="${prefix}base_footprint"></link>
+        <!-- BASE LINK -->
+        <link name="${prefix}base_link">
+            <visual>
+                <geometry>
+                    <mesh filename="file://$(find puzzlebot_description)/meshes/Puzzlebot_Jetson_Lidar_Edition_Base.stl"/>
+                </geometry>
+                <material name="orange"/>
+            </visual>
+            <collision>
+                <origin xyz="0.0 0.0 0.0" rpy="0.0 0.0 0.0"/>
+                <geometry>
+                    <box size="0.2 0.16 0.0503"/>
+                </geometry>
+            </collision>
+            <inertial>
+                <mass value="0.351"/>
+                <xacro:box_inertia mass="0.351" x="0.2" y="0.16" z="0.0503"/>
+            </inertial>
+        </link>
+        <joint name="${prefix}base_link_joint" type="fixed">
+            <origin xyz="0.0 0.0 0.05" rpy="0.0 0.0 0.0"/>
+            <parent link="${prefix}base_footprint"/>
+            <child link="${prefix}base_link"/>
+        </joint>
+        <!-- LEFT WHEEL -->
+        <link name="${prefix}left_wheel_link">
+            <visual>
+                <origin rpy="1.57 0.0 0.0"/>
+                <geometry>
+                    <mesh filename="file://$(find puzzlebot_description)/meshes/Puzzlebot_Wheel.stl"/>
+                </geometry>
+                <material name="orange"/>
+            </visual>
+            <collision>
+            <origin rpy="1.5707 0.0 0.0"/>
+                <geometry>
+                    <cylinder radius="0.05" length="0.012"/>
+                </geometry>
+            </collision>
+            <inertial>
+                <mass value="0.027"/>
+                <xacro:cylinder_inertia radius="0.05" height="0.012" mass="0.027"/>
+            </inertial>
+        </link>
+        <joint name="${prefix}left_wheel_joint" type="continuous">
+            <parent link="${prefix}base_link"/>
+            <child link="${prefix}left_wheel_link"/>
+            <origin xyz="0.052 0.095 -0.0025"/>
+            <axis xyz="0.0 1.0 0.0"/>
+        </joint>
+        <!-- RIGHT WHEEL -->
+        <link name="${prefix}right_wheel_link">
+            <visual>
+                <origin rpy="-1.57 0.0 0.0"/>
+                <geometry>
+                    <mesh filename="file://$(find puzzlebot_description)/meshes/Puzzlebot_Wheel.stl"/>
+                </geometry>
+                <material name="orange"/>
+            </visual>
+            <collision>
+            <origin rpy="1.5707 0.0 0.0"/>
+                <geometry>
+                    <cylinder radius="0.05" length="0.012"/>
+                </geometry>
+            </collision>
+            <inertial>
+                <mass value="0.027"/>
+                <xacro:cylinder_inertia radius="0.05" height="0.012" mass="0.027"/>
+            </inertial>
+        </link>
+        <joint name="${prefix}right_wheel_joint" type="continuous">
+            <parent link="${prefix}base_link"/>
+            <child link="${prefix}right_wheel_link"/>
+            <origin xyz="0.052 -0.095 -0.0025"/>
+            <axis xyz="0.0 1.0 0.0"/>
+        </joint>
+        <!-- CASTER  WHEEL -->
+        <link name="${prefix}caster_link">
+            <visual>
+                <origin xyz="0.0 0.0 -0.015"/>
+                <geometry>
+                    <mesh filename="file://$(find puzzlebot_description)/meshes/Puzzlebot_Caster_Wheel.stl"/>
+                </geometry>
+                <material name="orange"/>
+            </visual>
+            <collision>
+                <geometry>
+                    <sphere radius="0.02"/>
+                </geometry>
+            </collision>
+            <inertial>
+                <mass value="0.016"/>
+                <xacro:solid_sphere_inertia  mass="0.016" radius="0.02"/>
+            </inertial>
+        </link>
+        <joint name="${prefix}caster_joint" type="fixed">
+            <parent link="${prefix}base_link"/>
+            <child link="${prefix}caster_link"/>
+            <origin xyz="-0.095 0.0 -0.03"/>
+        </joint>
+    </xacro:macro>
 </robot>
